Commit message: added common properties and inerital properties to display model in gazebo

File: parrot_v1_description/urdf/common_properties.urdf.xacro (robot description, xacro)
@@ -1,12 +1,39 @@
 <?xml version="1.0"?>
-<robot xmlns:xacro="http://www.ros.org/wiki/xacro" >
-    <!-- <xacro:macro name="inertial" params="m xyz rpy" >
+<robot xmlns:xacro="http://www.ros.org/wiki/xacro">
+    <material name="blue">
+        <color rgba="0 0 0.5 0.5" />
+    </material>
+    <material name="green">
+        <color rgba="0 0.5 0 0.5" />
+    </material>
+    <material name="red">
+        <color rgba="0.5 0 0 0.5" />
+    </material>
+    <xacro:macro name="box_inertia" params="m l w h xyz rpy" >
         <inertial>
-            <origin xyz="${xyz}" rpy="${rpy}"/>
+            <origin xyz="${xyz}" rpy="${rpy}" />
             <mass value="${m}"  />
-            <inertia ixx="1.0" ixy="0.0" ixz="0.0"
-                     iyy="1.0" iyz="0.0"
-                     izz="1.0"/>
+            <inertia ixx="${(m/12) * (h*h + l*l)}" ixy="0.0" ixz="0.0"
+                     iyy="${(m/12) * (w*w + l*l)}" iyz="0.0"
+                     izz="${(m/12) * (w*w + h*h)}"/>
         </inertial>
-    </xacro:macro> -->
+    </xacro:macro>
+    <xacro:macro name="cylinder_inertia" params="m r h xyz rpy" >
+        <inertial>
+            <origin xyz="${xyz}" rpy="${rpy}" />
+            <mass value="${m}"  />
+            <inertia ixx="${(m/12) * (3*r*r + h*h)}" ixy="0.0" ixz="0.0"
+                     iyy="${(m/12) * (3*r*r + h*h)}" iyz="0.0"
+                     izz="${(m/2) * (r*r)}"/>
+        </inertial>
+    </xacro:macro>
+    <xacro:macro name="sphere_inertia" params="m r xyz rpy" >
+        <inertial>
+            <origin xyz="${xyz}" rpy="${rpy}" />
+            <mass value="${m}"  />
+            <inertia ixx="${2/5 * (m * r * r)}" ixy="0.0" ixz="0.0"
+                     iyy="${2/5 * (m * r * r)}" iyz="0.0"
+                     izz="${2/5 * (m * r * r)}"/>
+        </inertial>
+    </xacro:macro>
 </robot>

File: parrot_v1_description/urdf/parrot_v1.urdf.xacro (robot description, xacro)
@@ -2,7 +2,8 @@
 <robot xmlns:xacro="http://www.ros.org/wiki/xacro" >
     <!-- All dimensions multiplied by a factor of 10 for simulation -->
-    <xacro:property name="bp_length" value="0.067" />
-    <xacro:property name="bp_width" value="0.143" />
-    <xacro:property name="bp_height" value="0.0425" />
+    <!-- <box size="0.067 0.143 0.0425"/>    -->
+    <xacro:property name="bp_length" value="0.67" />
+    <xacro:property name="bp_width" value="1.43" />
+    <xacro:property name="bp_height" value="0.425" />
     <link name="base_footprint_v1" />
     <link name="base_parrot">
@@ -10,14 +11,25 @@
             <geometry>
                 <!-- Original Dimensions -->
-                <!-- <box size="0.067 0.143 0.0425"/>    -->
-                <box size="${10 * bp_length} ${10 * bp_width} ${10 * bp_height}"/>
+                <box size="${bp_length} ${bp_width} ${bp_height}"/>
             </geometry>
             <origin xyz="0.0 0.0 0.0" rpy="0.0 0.0 0.0"/>
+            <material name="green"/>
         </visual>
+        <collision>
+            <geometry>
+                <!-- Original Dimensions -->
+                <!-- <box size="0.067 0.143 0.0425"/>    -->
+                <box size="${bp_length} ${bp_width} ${bp_height}"/>
+            </geometry>
+            <origin xyz="0.0 0.0 0.0" rpy="0.0 0.0 0.0"/>
+        </collision>
+        <xacro:box_inertia m="1.0"
+                           l="${bp_length}" w="${bp_width}" h="${bp_height}"
+                           xyz="0 0 0" rpy="0 0 0" />
     </link>
     <joint name="base_footprint_link_joint" type="fixed">
         <parent link="base_footprint_v1"/>
         <child link="base_parrot"/>
-        <origin xyz="0 0 ${(bp_height * 10) /2}" rpy="0.0 0.0 0.0"/>
+        <origin xyz="0 0 ${bp_height /2}" rpy="0.0 0.0 0.0"/>
     </joint>
 </robot>
