Commit message: model simulated in gazebo, gripper contruction not done yet

File: parrot_v1_description/urdf/parrot_v1.urdf.xacro (robot description, xacro)
@@ -6,4 +6,25 @@
     <xacro:property name="bp_width" value="1.43" />
     <xacro:property name="bp_height" value="0.425" />
+    <!-- Link 1 -->
+    <xacro:property name="l1_radius" value="0.35" />
+    <xacro:property name="l1_height" value="0.04" />
+    <!-- Link 1 and 2 offset -->
+    <xacro:property name="l12_offset" value="0.3925" />
+    <!-- Link 2 and 3 offset -->
+    <xacro:property name="l23_offset" value="0.674" />
+    <!-- Link 2 -->
+    <xacro:property name="l2_length" value="0.452" />
+    <xacro:property name="l2_width" value="0.243" />
+    <xacro:property name="l2_height" value="1.115" />
+    <!-- Link 3 -->
+    <xacro:property name="l3_length" value="0.48" />
+    <xacro:property name="l3_width" value="0.20" />
+    <xacro:property name="l3_height" value="0.404" />
+    <!-- Link 4 -->
+    <xacro:property name="l4_length" value="0.56" />
+    <xacro:property name="l4_width" value="0.20" />
+    <xacro:property name="l4_height" value="0.20" />
+    <xacro:property name="effort" value="30"/>
+    <xacro:property name="velocity" value="10"/>
     <link name="base_footprint_v1" />
     <link name="base_parrot">
@@ -19,5 +40,4 @@
             <geometry>
                 <!-- Original Dimensions -->
-                <!-- <box size="0.067 0.143 0.0425"/>    -->
                 <box size="${bp_length} ${bp_width} ${bp_height}"/>
             </geometry>
@@ -28,4 +48,75 @@
                            xyz="0 0 0" rpy="0 0 0" />
     </link>
+    <link name="link_1">
+        <visual>
+            <geometry>
+                <cylinder radius="${l1_radius}" length="${l1_height}"/>
+            </geometry>
+            <origin xyz="0 0 0" rpy="0 0 0"/>
+            <material name="red"/>
+        </visual>
+        <collision>
+            <geometry>
+                <cylinder radius="${l1_radius}" length="${l1_height}"/>
+            </geometry>
+            <origin xyz="0 0 0" rpy="0 0 0"/>
+        </collision>
+        <xacro:cylinder_inertia m="1.0" r="${l1_radius}  " h="${l1_height}"
+                           xyz="0 0 0" rpy="0 0 0" />
+    </link>
+    <link name="link_2">
+        <visual>
+            <geometry>
+                <box size="${l2_length} ${l2_width} ${l2_height}"/>
+            </geometry>
+            <origin xyz="0 0 ${l2_height/2 - 0.2205}" rpy="0 0 0"/>
+            <material name="green"/>
+        </visual>
+        <collision>
+            <geometry>
+                <box size="${l2_length} ${l2_width} ${l2_height}"/>
+            </geometry>
+            <origin xyz="0 0 ${l2_height/2 - 0.2205}" rpy="0 0 0"/>
+        </collision>
+        <xacro:box_inertia m="1.0"
+                           l="${l2_length}" w="${l2_width}" h="${l2_height}"
+                           xyz="0 0 0" rpy="0 0 0" />
+    </link>
+    <link name="link_3">
+        <visual>
+            <geometry>
+                <box size="${l3_length} ${l3_width} ${l3_height}"/>
+            </geometry>
+            <origin xyz="0 0 0.674" rpy="0 0 0"/>
+            <material name="red"/>
+        </visual>
+        <collision>
+            <geometry>
+                <box size="${l3_length} ${l3_width} ${l3_height}"/>
+            </geometry>
+            <origin xyz="0 0 0.674" rpy="0 0 0"/>
+        </collision>
+        <xacro:box_inertia m="1.0"
+                           l="${l3_length}" w="${l3_width}" h="${l3_height}"
+                           xyz="0 0 0" rpy="0 0 0" />
+    </link>
+    <link name="link_4">
+        <visual>
+            <geometry>
+                <box size="${l4_length} ${l4_width} ${l4_height}"/>
+            </geometry>
+            <origin xyz="0 0 0.5603" rpy="0 0 0"/>
+            <material name="green"/>
+        </visual>
+        <collision>
+            <geometry>
+                <box size="${l4_length} ${l4_width} ${l4_height}"/>
+            </geometry>
+            <origin xyz="0 0 0.5603" rpy="0 0 0"/>
+        </collision>
+        <xacro:box_inertia m="1.0"
+                           l="${l4_length}" w="${l4_width}" h="${l4_height}"
+                           xyz="0 0 0" rpy="0 0 0" />
+    </link>
     <joint name="base_footprint_link_joint" type="fixed">
         <parent link="base_footprint_v1"/>
@@ -33,3 +124,31 @@
         <origin xyz="0 0 ${bp_height /2}" rpy="0.0 0.0 0.0"/>
     </joint>
+    <joint name="base_j1_joint" type="revolute">
+        <parent link="base_parrot"/>
+        <child link="link_1"/>
+        <origin xyz="0 0 ${bp_height/2 + l1_height/2}" rpy="0 0 0"/>
+        <axis xyz="0 0 1"/>
+        <limit lower="${pi /2}" upper="${-pi /2}" effort="${effort}" velocity="${velocity}"/>
+    </joint>
+    <joint name="link_1_2_joint" type="revolute">
+        <parent link="link_1"/>
+        <child link="link_2"/>
+        <origin xyz="0 0 0${l1_height/2 + l12_offset}" rpy="0 0 0"/>
+        <axis xyz="1 0 0"/>
+        <limit lower="${pi /2}" upper="${-pi /2}" effort="${effort}" velocity="${velocity}"/>
+    </joint>
+    <joint name="link_2_3_joint" type="revolute">
+        <parent link="link_2"/>
+        <child link="link_3"/>
+        <origin xyz="0 0 0.674" rpy="0 0 0"/>
+        <axis xyz="1 0 0"/>
+        <limit lower="${pi /2}" upper="${-pi /2}" effort="${effort}" velocity="${velocity}"/>
+    </joint>
+    <joint name="link_3_4_joint" type="revolute">
+        <parent link="link_3"/>
+        <child link="link_4"/>
+        <origin xyz="0 0 0.674" rpy="0 0 0"/>
+        <axis xyz="1 0 0"/>
+        <limit lower="${pi /2}" upper="${-pi /2}" effort="${effort}" velocity="${velocity}"/>
+    </joint>
 </robot>

File: parrot_v1_description/urdf/parrot_v1_main.urdf.xacro (robot description, xacro)
@@ -3,4 +3,4 @@
     <xacro:include filename="common_properties.urdf.xacro" />
     <xacro:include filename="parrot_v1.urdf.xacro" />
-    <!-- <xacro:include filename="parrot_v1_simple.urdf" />     -->
+    <xacro:include filename="parrot_v1_gazebo.urdf.xacro" />
 </robot>

Commit message: added parrot_v1_controller and its components

File: parrot_v1_description/urdf/parrot_v1.urdf.xacro (robot description, xacro)
@@ -124,5 +124,5 @@
         <origin xyz="0 0 ${bp_height /2}" rpy="0.0 0.0 0.0"/>
     </joint>
-    <joint name="base_j1_joint" type="revolute">
+    <joint name="joint_1" type="revolute">
         <parent link="base_parrot"/>
         <child link="link_1"/>
@@ -131,5 +131,5 @@
         <limit lower="${pi /2}" upper="${-pi /2}" effort="${effort}" velocity="${velocity}"/>
     </joint>
-    <joint name="link_1_2_joint" type="revolute">
+    <joint name="joint_2" type="revolute">
         <parent link="link_1"/>
         <child link="link_2"/>
@@ -138,5 +138,5 @@
         <limit lower="${pi /2}" upper="${-pi /2}" effort="${effort}" velocity="${velocity}"/>
     </joint>
-    <joint name="link_2_3_joint" type="revolute">
+    <joint name="joint_3" type="revolute">
         <parent link="link_2"/>
         <child link="link_3"/>
@@ -145,5 +145,5 @@
         <limit lower="${pi /2}" upper="${-pi /2}" effort="${effort}" velocity="${velocity}"/>
     </joint>
-    <joint name="link_3_4_joint" type="revolute">
+    <joint name="joint_4" type="revolute">
         <parent link="link_3"/>
         <child link="link_4"/>
@@ -152,3 +152,16 @@
         <limit lower="${pi /2}" upper="${-pi /2}" effort="${effort}" velocity="${velocity}"/>
     </joint>
+    <xacro:macro name="default_transmission" params="suffix" >
+        <transmission name="transmission_${suffix}">
+            <plugin>transmission_interface/SimpleTransmission</plugin>
+            <actuator name="motor_${suffix}" />
+            <joint name="$joint_${suffix}" >
+                <mechanical_reduction>1.0</mechanical_reduction>
+            </joint>
+        </transmission>
+    </xacro:macro>
+    <xacro:default_transmission suffix="1" />
+    <xacro:default_transmission suffix="2" />
+    <xacro:default_transmission suffix="3" />
+    <xacro:default_transmission suffix="4" />
 </robot>

File: parrot_v1_description/urdf/parrot_v1_gazebo.urdf.xacro (robot description, xacro)
@@ -1,28 +1,10 @@
 <?xml version="1.0"?>
 <robot xmlns:xacro="http://www.ros.org/wiki/xacro" name="robot_name">
-    <gazebo reference="base_parrot">
-        <material>
-            Gazebo/Blue
-        </material>
-    </gazebo>
-    <gazebo reference="link_1">
-        <material>
-            Gazebo/Blue
-        </material>
-    </gazebo>
-    <gazebo reference="link_2">
-        <material>
-            Gazebo/Blue
-        </material>
-    </gazebo>
-    <gazebo reference="link_3">
-        <material>
-            Gazebo/Blue
-        </material>
-    </gazebo>
-    <gazebo reference="link_5">
-        <material>
-            Gazebo/Blue
-        </material>
+    <gazebo>
+        <plugin filename="libgazebo_ros2_control.so" name="gazebo_ros2_control">
+            <robot_param>robot_description</robot_param>
+            <robot_param_node>robot_state_publisher</robot_param_node>
+            <parameters>$(find parrot_v1_controller)/config/parrot_v1_control.yaml</parameters>
+        </plugin>
     </gazebo>
 </robot>

File: parrot_v1_description/urdf/parrot_v1_main.urdf.xacro (robot description, xacro)
@@ -4,3 +4,4 @@
     <xacro:include filename="parrot_v1.urdf.xacro" />
     <xacro:include filename="parrot_v1_gazebo.urdf.xacro" />
+    <xacro:include filename="parrot_v1_control.xacro" />
 </robot>

Commit message: added new packages - the parrot_v1 - moveit, msgs, utils, examples and added new launch files in moveit and bringup

File: parrot_v1_description/urdf/parrot_v1.urdf.xacro (robot description, xacro)
@@ -119,5 +119,5 @@
                            xyz="0 0 0" rpy="0 0 0" />
     </link>
-    <joint name="base_footprint_link_joint" type="fixed">
+    <joint name="root_joint" type="fixed">
         <parent link="base_footprint_v1"/>
         <child link="base_parrot"/>

Commit message: added parrot Firware package to make the arduino ros bridge

File: parrot_v1_description/urdf/parrot_v1.urdf.xacro (robot description, xacro)
@@ -119,5 +119,5 @@
                            xyz="0 0 0" rpy="0 0 0" />
     </link>
-    <joint name="root_joint" type="fixed">
+    <joint name="virtual_joint" type="fixed">
         <parent link="base_footprint_v1"/>
         <child link="base_parrot"/>

File: parrot_v1_description/urdf/parrot_v1_main.urdf.xacro (robot description, xacro)
@@ -4,4 +4,4 @@
     <xacro:include filename="parrot_v1.urdf.xacro" />
     <xacro:include filename="parrot_v1_gazebo.urdf.xacro" />
-    <xacro:include filename="parrot_v1_control.xacro" />
+    <!-- <xacro:include filename="parrot_v1_control.xacro" />     -->
 </robot>
